File: v1/KicadProj/raylar_v1_00/Sheet2.kicad_sch (KiCad schematic)
At the start: 41 parts, among them J1 3.5mm, J2 3.5mm, J3 USB_C_Receptacle, J4 B2B-PH-SM4-TB, U2 TPS629210DRLR, U3 BQ25186, U4 TLV75733PDRV

Commit message: Updated fab
Parts:
- C17, C20, C21, C22, C23, C24: Q_SUPPLIER (none) -> QUICK-TECK; Q_SUPPLIER_PN (none) -> QCC-00295
- C18, C19, C25, C27: Q_SUPPLIER (none) -> QUICK-TECK; Q_SUPPLIER_PN (none) -> QCC-00426
- C26: Q_SUPPLIER (none) -> QUICK-TECK; Q_SUPPLIER_PN (none) -> QCC-00294
- D1, D2, D3, D4, D5: MP MBR0530T1G -> MBR130T1G; Q_SUPPLIER (none) -> LCSC; Q_SUPPLIER_PN (none) -> C82461; Voltage (none) -> 30V
- J1, J2: Q_SUPPLIER (none) -> LCSC; Q_SUPPLIER_PN (none) -> C695629
- J3: Q_SUPPLIER (none) -> LCSC; Q_SUPPLIER_PN (none) -> C2988369
- J4: Q_SUPPLIER (none) -> LCSC; Q_SUPPLIER_PN (none) -> C160352
- L2: Q_SUPPLIER (none) -> LCSC; Q_SUPPLIER_PN (none) -> C237482
- R10, R12, R9: Q_SUPPLIER (none) -> LCSC; Q_SUPPLIER_PN (none) -> C25905
- R11: Q_SUPPLIER (none) -> LCSC; Q_SUPPLIER_PN (none) -> C276270
- R13, R15: Q_SUPPLIER (none) -> QUICK-TECK; Q_SUPPLIER_PN (none) -> QCR-00076
- R14: Q_SUPPLIER (none) -> QUICK-TECK; Q_SUPPLIER_PN (none) -> QCR-00098
- R16, R17, R4, R6: Q_SUPPLIER (none) -> QUICK-TECK; Q_SUPPLIER_PN (none) -> QCR-00086
- R3, R5: Q_SUPPLIER (none) -> QUICK-TECK; Q_SUPPLIER_PN (none) -> QCR-00102
- R7, R8: Q_SUPPLIER (none) -> QUICK-TECK; Q_SUPPLIER_PN (none) -> QCR-00018
- U2: Q_SUPPLIER (none) -> MOUSER; Q_SUPPLIER_PN (none) -> 595-TPS629210DRLR
- U3: Q_SUPPLIER (none) -> MOUSER; Q_SUPPLIER_PN (none) -> 595-BQ25186DLHR
- U4: Q_SUPPLIER (none) -> MOUSER; Q_SUPPLIER_PN (none) -> 595-TLV75733PDRVR
