File: v1/KicadProj/raylar_v1_00/sheet1.kicad_sch (KiCad schematic)
At the start: 27 parts, among them SW1 SMD_4.6x2.8mm, SW2 SMD_4.6x2.8mm, U1 STM32U5G7VJTxQ, Y1 ABM8AIG-16.000MHZ-12-2Z-T3, Y2 32.768kHz ABS07-32.768KHZ-T

Commit message: Updated fab
Parts:
- C1, C2, C4, C5, C6: Q_SUPPLIER (none) -> QUICK-TECK; Q_SUPPLIER_PN (none) -> QCC-00294
- C10, C11, C16, C3, C7, C8, C9: Q_SUPPLIER (none) -> QUICK-TECK; Q_SUPPLIER_PN (none) -> QCC-00426
- C12, C13, C14, C15: Q_SUPPLIER (none) -> QUICK-TECK; Q_SUPPLIER_PN (none) -> QCC-00384
- L1: Q_SUPPLIER (none) -> LCSC; Q_SUPPLIER_PN (none) -> C237482
- R1, R2: Q_SUPPLIER (none) -> QUICK-TECK; Q_SUPPLIER_PN (none) -> QCR-00076
- SW1, SW2: Q_SUPPLIER (none) -> LCSC; Q_SUPPLIER_PN (none) -> C221676
- U1: value STM32U5G7VJTxQ -> STM32U595VJT6Q; Q_SUPPLIER (none) -> MOUSER; Q_SUPPLIER_PN (none) -> 511-STM32U595VJT6Q
- Y1: Q_SUPPLIER (none) -> LCSC; Q_SUPPLIER_PN (none) -> C596903
- Y2: Q_SUPPLIER (none) -> LCSC; Q_SUPPLIER_PN (none) -> C130253
