File: v1/KicadProj/raylar_v1_00/sheet3.kicad_sch (KiCad schematic)
At the start: 35 parts, among them J5 microSD, U5 E80-900M2213S, U6 FDV304P, U7 L86-M33

Commit message: Updated fab
Parts:
- C28, C30, C31, C33, C35: Q_SUPPLIER (none) -> QUICK-TECK; Q_SUPPLIER_PN (none) -> QCC-00294
- C29, C32, C34, C36: Q_SUPPLIER (none) -> QUICK-TECK; Q_SUPPLIER_PN (none) -> QCC-00426
- D10: Q_SUPPLIER (none) -> QUICK-TECK; Q_SUPPLIER_PN (none) -> QCD-00048
- D8: Q_SUPPLIER (none) -> QUICK-TECK; Q_SUPPLIER_PN (none) -> QCD-00046
- D9: Q_SUPPLIER (none) -> QUICK-TECK; Q_SUPPLIER_PN (none) -> QCD-00045
- J5: Q_SUPPLIER (none) -> LCSC; Q_SUPPLIER_PN (none) -> C20619272
- R18, R19, R20, R23, R24, R26: Q_SUPPLIER (none) -> QUICK-TECK; Q_SUPPLIER_PN (none) -> QCR-00086
- R25, R29, R30: Q_SUPPLIER (none) -> LCSC; Q_SUPPLIER_PN (none) -> C25879
- R27: Q_SUPPLIER (none) -> QUICK-TECK; Q_SUPPLIER_PN (none) -> QCR-00098
- R28: Q_SUPPLIER (none) -> QUICK-TECK; Q_SUPPLIER_PN (none) -> QCR-00042
- U5: Q_SUPPLIER (none) -> LCSC; Q_SUPPLIER_PN (none) -> C42464134
- U6: Q_SUPPLIER (none) -> LCSC; Q_SUPPLIER_PN (none) -> C5219301
- U7: Q_SUPPLIER (none) -> LCSC; Q_SUPPLIER_PN (none) -> C909689
