File: v1/KicadProj/raylar_v1_00/sheet4.kicad_sch (KiCad schematic)
At the start: 30 parts, among them U8 LIS2HH12, U9 LIS2MDL

Commit message: Updated fab
Parts:
- C37, C38, C39, C41, C42, C43, C53: Q_SUPPLIER (none) -> QUICK-TECK; Q_SUPPLIER_PN (none) -> QCC-00294
- C40, C44, C45, C46, C47, C48, C49, C50, C51, C52: Q_SUPPLIER (none) -> QUICK-TECK; Q_SUPPLIER_PN (none) -> QCC-00426
- MK1, MK2, MK3, MK4, MK5, MK6: Q_SUPPLIER (none) -> MOUSER; Q_SUPPLIER_PN (none) -> 726-IM69D129FV01XTMA
- R31, R32: Q_SUPPLIER (none) -> QUICK-TECK; Q_SUPPLIER_PN (none) -> QCR-00076
- U8: Q_SUPPLIER (none) -> LCSC; Q_SUPPLIER_PN (none) -> C221446
- U9: Q_SUPPLIER (none) -> LCSC; Q_SUPPLIER_PN (none) -> C919695
