File: v1/KicadProj/raylar_v1_00/sheet5.kicad_sch (KiCad schematic)
At the start: 16 parts, among them J10 Conn_01x08, J6 Conn_01x08, J7 Qwiic_RA, J8 Qwiic_RA, J9 89898-308ALF, SW3 SMD_4.6x2.8mm, U10 CPT-9019A-SMT-TR

Commit message: Updated fab
Parts:
- C54: Q_SUPPLIER (none) -> QUICK-TECK; Q_SUPPLIER_PN (none) -> QCC-00426
- D11: Q_SUPPLIER (none) -> QUICK-TECK; Q_SUPPLIER_PN (none) -> QCD-00045
- D12: Q_SUPPLIER (none) -> QUICK-TECK; Q_SUPPLIER_PN (none) -> QCD-00048
- J10, J6: Q_SUPPLIER (none) -> MOUSER; Q_SUPPLIER_PN (none) -> 640-BG125-8A1144ND
- J7, J8: Q_SUPPLIER (none) -> LCSC; Q_SUPPLIER_PN (none) -> C160404
- J9: Q_SUPPLIER (none) -> LCSC; Q_SUPPLIER_PN (none) -> C5417482
- R33, R34, R38: Q_SUPPLIER (none) -> QUICK-TECK; Q_SUPPLIER_PN (none) -> QCR-00076
- R35: Q_SUPPLIER (none) -> QUICK-TECK; Q_SUPPLIER_PN (none) -> QCR-00018
- R36, R37: Q_SUPPLIER (none) -> LCSC; Q_SUPPLIER_PN (none) -> C25879
- SW3: Q_SUPPLIER (none) -> LCSC; Q_SUPPLIER_PN (none) -> C221676
- U10: Q_SUPPLIER (none) -> MOUSER; Q_SUPPLIER_PN (none) -> 179-CPT-9019A-SMT-TR
